File: Airdahl 1.0/sensors.kicad_sch (KiCad schematic)
At the start: 32 parts, among them J10 Conn_01x06_Pin, J6 PRT-16766, J7 CONUFL001-SMD-T, J9 104031-0811, U3 ADXL345, U4 BNO085, U5 BMP581, U6 RFM95W-915S2

Commit message: restructured airdahl for carrier boards, switched 20 pin debug jtag for 10 pin for use with adafruit usb stlink, schematic formatting
Parts:
- removed C8, C9: 100n, Capacitor_SMD:C_0603_1608Metric_Pad1.08x0.95mm_HandSolder, symbol Device:C_Small
- removed J10: Conn_01x06_Pin, Connector_PinSocket_2.54mm:PinSocket_1x06_P2.54mm_Vertical, symbol Connector:Conn_01x06_Pin
- removed J6: PRT-16766, CONN_BM04B-SRSS-TB_SPK, symbol 2025-12-12_19-35-05:PRT-16766
- removed U3: ADXL345, ADXL345:PQFN80P500X300X100-14N, symbol ADXL345:ADXL345
Connections:
- no-connect marks 11 -> 9
Other:
- note removed: "QWIIC I2C"
- note removed: "SPI Breakout"
- note removed: "Secondary IMU"
- company: (none) -> Washington University in St. Louis
- title: AirDahl Flight Computer -> AirDahl Flight Computer Primary Sensors

Commit message: added led and others
Connections:
- net CS_RFM: no longer J9.2 (CD/DAT3), R30.1
- new net CS_SD: J9.2 (CD/DAT3), R30.1
Changed lines of the file:
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@@
 		)
 	)
-	(hierarchical_label "CS_RFM"
+	(hierarchical_label "CS_SD"
 		(shape input)
 		(at 180.34 48.26 0)

Commit message: added to carrier board port pinout, need to add to mcu
Parts:
- added R52: 10k, Resistor_SMD:R_0402_1005Metric, symbol Device:R
Connections:
- net +3V3: now also R52.2
- net GND: now also J9.10 (SW-2)
- net CD: now reaches J9.9 (SW-1)
- net CD: now also R52.1
- no-connect marks 9 -> 7
