File: Airdahl 1.0/sensors.kicad_sch (KiCad schematic)
At the start: 28 parts, among them J7 CONUFL001-SMD-T, J9 104031-0811, U4 BNO085, U5 BMP581, U6 RFM95W-915S2

Commit message: stoning my cap
Parts:
- removed R28: 5.1k, Resistor_SMD:R_0402_1005Metric, symbol Device:R
- removed R29, R30, R31, R32, R38: 10k, Resistor_SMD:R_0402_1005Metric, symbol Device:R
- removed R39: 22, Resistor_SMD:R_0402_1005Metric, symbol Device:R
- added R53, R54, R55, R56, R57: 51k, Resistor_SMD:R_0402_1005Metric, symbol Device:R
Connections:
- net +3V3: now also R53.2, R54.2, R55.2, R56.2, R57.2
- net MOSI: no longer J9.3 (CMD)
- net SCLK: no longer J9.5 (CLK)
- net SDIO_D0: now reaches J9.7 (DAT0)
- net SDIO_D0: now also R54.1
- net SDIO_D2: now reaches J9.1 (DAT2)
- net SDIO_D2: now also R56.1
- net SDIO_D1: now reaches J9.8 (DAT1)
- net SDIO_D1: now also R55.1
- net CS_SD renamed SDIO_D3
- net SDIO_D3: now also R57.1
- new net SDIO_CLK: J9.5 (CLK)
- new net SDIO_CMD: J9.3 (CMD), R53.1
Other:
- moved on the sheet: C17, R52
