File: Airdahl 1.0/_restore_backup_2026-09-18T12-19-39-022/Airdahl 1.0.kicad_sch (KiCad schematic)
At the start: 67 parts, among them J1 Conn_01x04, J2 DF40C-34DS-0.4V_58_, J3 DF40C-34DS-0.4V_58_, J4 USB_C_Receptacle_USB2.0_16P, SW1 SW_SPST, SW2 SW_SPST, U1 STM32F446RETx, U2 MCP2200-I-MQ, U7 NCP1117-3.3_SOT223, Y1 ABM3B-8.000MHZ-12-D1X-T, Y2 ABS25-32.768KHZ-6-T, Y3 12MHz

Commit message: routing changes
Parts:
- C37: value 330n -> 100n
Connections:
- net PA12 is gone; now on net RST_RFM: U1.45 (PA12)
- net PA15 is gone; now on net D0_RFM: U1.50 (PA15)
- net +3V3_REG: now also J3.8; no longer J3.12
- net BMP_INT: now also U1.58 (PB6)
- net BNO_INT: now also U1.16 (PA2)
- net BNO_RST: now also U1.15 (PA1)
- net GND: now also J3.31, J3.33; no longer J3.32, J3.34
- net PA0: now also J2.31; no longer J3.4
- net PA1: now also J2.29; no longer J3.6, U1.15 (PA1)
- net PA2: now also J2.16; no longer J3.8, U1.16 (PA2)
- net PA3: now also J3.17; no longer J3.5
- net PAYLOAD_1F: now also J2.14; no longer J2.16
- net PAYLOAD_1R: now also J2.12; no longer J2.14
- net PB6: no longer U1.58 (PB6)
- net PC5: now also J3.27; no longer J2.20
- net PYRO_1: now also J2.22, U1.35 (PB14); no longer J3.33, U1.36 (PB15)
- net PYRO_2: now also J2.24, U1.34 (PB13); no longer J3.31, U1.35 (PB14)
- net PYRO_3: now also J2.26, U1.33 (PB12); no longer J3.29, U1.34 (PB13)
- net PYRO_4: now also J3.25, U1.29 (PB10); no longer J3.27, U1.33 (PB12)
- net PYRO_5: now also J2.20, U1.36 (PB15); no longer J3.25, U1.29 (PB10)
- net UART_RX: now also J3.3; no longer J3.17
- net UART_TX: now also J3.5; no longer J3.19
Other:
- note added: "V_REG on carrier boards"
- note added: "X Put UART_RX on MCU pin, make sure it's UART1 X Make sure it's RX -> TX, TX -> RX X Find new Payload Reverse IO Find more IO's for SPI CS X one more pyro channel HIGH: find a lower fwd voltage schottky diode bonus: battery charge indicator"
- note removed: "V_REG is a voltage (3V3) on carrier boards USB_3V3 is generated on the main board after the USB port, it's VBUS stepped down SWD_3V3 would come from the ST Link"
- note removed: "X Put UART_RX on MCU pin, make sure it's UART1 X Make sure it's RX -> TX, TX -> RX X Find new Payload Reverse IO Find more IO's for SPI CS X one more pyro channel BNO_RST doesn't go anywhere BNO_INT doesn't go anywhere HIGH: replace schottky diode or-ing with ideal diodes, or power mux Check if UART and SDIO conflict bonus: battery charge indicator"
