File: Airdahl 1.0/_restore_backup_2026-09-18T12-19-39-022/sensors.kicad_sch (KiCad schematic)
At the start: 27 parts, among them J7 CONUFL001-SMD-T, J9 104031-0811, U4 BNO085, U5 BMP581, U6 RFM95W-915S2

Commit message: routing changes
Parts:
- added C18: 100n, Capacitor_SMD:C_0402_1005Metric, symbol Device:C
- C13: value 10n -> 10u
- C17: value 1u -> 10u; footprint Capacitor_SMD:C_0402_1005Metric -> Capacitor_SMD:C_0805_2012Metric
Connections:
- net +3V3: now also C18.1
- net GND: now also C18.2
Changed lines of the file:
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@@
 	)
 	(junction
+		(at 137.16 40.64)
+		(diameter 0)
+		(color 0 0 0 0)
+	)
+	(junction
 		(at 118.11 69.85)
 		(diameter 0)
@@
 	)
 	(junction
+		(at 137.16 48.26)
+		(diameter 0)
+		(color 0 0 0 0)
+	)
+	(junction
 		(at 124.46 184.15)
 		(diameter 0)
@@
 	(wire
 		(pts
+			(xy 124.46 48.26) (xy 137.16 48.26)
+		)
+		(stroke
+			(width 0)
+			(type default)
+		)
+	)
+	(wire
+		(pts
 			(xy 119.38 163.83) (xy 135.89 163.83)
 		)
@@
 	(wire
 		(pts
+			(xy 124.46 40.64) (xy 137.16 40.64)
+		)
+		(stroke
+			(width 0)
+			(type default)
+		)
+	)
+	(wire
+		(pts
 			(xy 26.67 148.59) (xy 29.21 148.59)
 		)
@@
 	(wire
 		(pts
-			(xy 124.46 39.37) (xy 124.46 40.64)
+			(xy 124.46 67.31) (xy 110.49 67.31)
 		)
 		(stroke
@@
 	(wire
 		(pts
-			(xy 124.46 67.31) (xy 110.49 67.31)
+			(xy 26.67 173.99) (xy 26.67 148.59)
 		)
 		(stroke
@@
 	(wire
 		(pts
-			(xy 26.67 173.99) (xy 26.67 148.59)
+			(xy 40.64 163.83) (xy 58.42 163.83)
 		)
 		(stroke
@@
 	(wire
 		(pts
-			(xy 40.64 163.83) (xy 58.42 163.83)
+			(xy 137.16 39.37) (xy 137.16 40.64)
 		)
 		(stroke
@@
 			)
 		)
-		(property "Value" "10n"
+		(property "Value" "10u"
 			(at 274.32 97.7962 0)
 			(show_name no)
@@
 	(symbol
 		(lib_id "power:+3V3")
-		(at 124.46 39.37 0)
+		(at 137.16 39.37 0)
 		(unit 1)
 		(body_style 1)
@@
 		(fields_autoplaced yes)
 		(property "Reference" "#PWR070"
-			(at 124.46 43.18 0)
+			(at 137.16 43.18 0)
 			(hide yes)
 			(show_name no)
@@
 		)
 		(property "Value" "+3V3"
-			(at 124.46 34.29 0)
+			(at 137.16 34.29 0)
 			(show_name no)
 			(do_not_autoplace no)
@@
 		)
 		(property "Footprint" ""
-			(at 124.46 39.37 0)
+			(at 137.16 39.37 0)
 			(hide yes)
 			(show_name no)
@@
 		)
 		(property "Datasheet" ""
-			(at 124.46 39.37 0)
+			(at 137.16 39.37 0)
 			(hide yes)
 			(show_name no)
@@
 		)
 		(property "Description" "Power symbol creates a global label with name \"+3V3\""
-			(at 124.46 39.37 0)
+			(at 137.16 39.37 0)
 			(hide yes)
 			(show_name no)
@@
 	(symbol
 		(lib_id "power:GND")
-		(at 124.46 48.26 0)
+		(at 137.16 48.26 0)
 		(unit 1)
 		(body_style 1)
@@
 		(fields_autoplaced yes)
 		(property "Reference" "#PWR071"
-			(at 124.46 54.61 0)
+			(at 137.16 54.61 0)
 			(hide yes)
 			(show_name no)
@@
 		)
 		(property "Value" "GND"
-			(at 124.46 53.34 0)
+			(at 137.16 53.34 0)
 			(show_name no)
 			(do_not_autoplace no)
@@
 		)
 		(property "Footprint" ""
-			(at 124.46 48.26 0)
+			(at 137.16 48.26 0)
 			(hide yes)
 			(show_name no)
@@
 		)
 		(property "Datasheet" ""
-			(at 124.46 48.26 0)
+			(at 137.16 48.26 0)
 			(hide yes)
 			(show_name no)
@@
 		)
 		(property "Description" "Power symbol creates a global label with name \"GND\" , ground"
-			(at 124.46 48.26 0)
+			(at 137.16 48.26 0)
 			(hide yes)
 			(show_name no)
@@
 			)
 		)
-		(property "Value" "1u"
+		(property "Value" "10u"
 			(at 128.27 46.482 0)
 			(show_name no)
@@
 			)
 		)
-		(property "Footprint" "Capacitor_SMD:C_0402_1005Metric"
+		(property "Footprint" "Capacitor_SMD:C_0805_2012Metric"
 			(at 125.4252 48.26 0)
 			(hide yes)
@@
 					(unit 1)
 				)
+			)
+		)
+	)
+	(symbol
+		(lib_id "Device:C")
+		(at 137.16 44.45 0)
+		(unit 1)
+		(body_style 1)
+		(exclude_from_sim no)
+		(in_bom yes)
+		(on_board yes)
+		(in_pos_files yes)
+		(dnp no)
+		(property "Reference" "C18"
+			(at 141.732 43.688 0)
+			(show_name no)
+			(do_not_autoplace no)
+			(effects
+				(font
+					(size 1.27 1.27)
+				)
+				(justify left)
+			)
+		)
+		(property "Value" "100n"
+			(at 140.97 46.482 0)
+			(show_name no)
+			(do_not_autoplace no)
+			(effects
+				(font
+					(size 1.27 1.27)
+				)
+				(justify left)
+			)
+		)
+		(property "Footprint" "Capacitor_SMD:C_0402_1005Metric"
+			(at 138.1252 48.26 0)
+			(hide yes)
+			(show_name no)
+			(do_not_autoplace no)
+			(effects
+				(font
+					(size 1.27 1.27)
+				)
+			)
+		)
+		(property "Datasheet" ""
+			(at 137.16 44.45 0)
+			(hide yes)
+			(show_name no)
+			(do_not_autoplace no)
+			(effects
+				(font
+					(size 1.27 1.27)
+				)
+			)
+		)
+		(property "Description" "Unpolarized capacitor"
+			(at 137.16 44.45 0)
+			(hide yes)
+			(show_name no)
+			(do_not_autoplace no)
+			(effects
+				(font
+					(size 1.27 1.27)
+				)
+			)
+		)
+		(pin "1"
+		)
+		(pin "2"
+		)
+		(instances
+			(project "Airdahl 1.0"
+				(path "/e2c992a5-0f37-48ff-88a4-7c40cfcda45e/bd752d91-9d5e-4749-819a-1163586784de"
+					(reference "C18")
+					(unit 1)
+				)
