File: Airdahl 1.0/_restore_backup_2026-09-19T19-26-46-477/Airdahl 1.0.kicad_pcb (KiCad board)
At the start: 2 copper layers, 57.6 x 39.5 mm, 94 parts, among them J1 Conn_01x04, J2 DF40C-34DS-0.4V_58_, J3 DF40C-34DS-0.4V_58_, J4 USB_C_Receptacle_USB2.0_16P, J7 CONUFL001-SMD-T, J9 104031-0811, SW1 SW_SPST, SW2 SW_SPST, U1 STM32F446RETx, U2 MCP2200-I-MQ, U4 BNO085, U5 BMP581, U6 RFM95W-915S2, U7 NCP1117-3.3_SOT223, Y1 ABM3B-8.000MHZ-12-D1X-T, Y2 ABS25-32.768KHZ-6-T, Y3 12MHz

Commit message: idk what i have but there are certainly changes
Parts:
- moved U6 15.8 mm to (215.9, 90.8)
- moved J9 11.2 mm to (211.1, 115.7)
- moved R53 7.16 mm to (188.9, 123.0)
- moved R54 3.52 mm to (187.9, 116.0)
- moved R57 2.61 mm to (186.9, 103.0)
- moved R55 2.08 mm to (187.9, 112.5)
Routing:
- net Net-(C33-Pad2): track 11.8 -> 10.5 mm
