File: Airdahl 1.0/_restore_backup_2026-09-22T14-01-29-934/Airdahl 1.0.kicad_pcb (KiCad board)
At the start: 2 copper layers, 57.6 x 39.5 mm, 94 parts, among them J1 Conn_01x04, J2 DF40C-34DS-0.4V_58_, J3 DF40C-34DS-0.4V_58_, J4 USB_C_Receptacle_USB2.0_16P, J7 CONUFL001-SMD-T, J9 104031-0811, SW1 SW_SPST, SW2 SW_SPST, U1 STM32F446RETx, U2 MCP2200-I-MQ, U4 BNO085, U5 BMP581, U6 RFM95W-915S2, U7 NCP1117-3.3_SOT223, Y1 ABM3B-8.000MHZ-12-D1X-T, Y2 ABS25-32.768KHZ-6-T, Y3 12MHz

Commit message: idk what i have but there are certainly changes
Parts:
- moved U6 15.8 mm to (215.9, 90.8)
- moved J9 11.2 mm to (211.1, 115.7)
- moved R53 7.16 mm to (188.9, 123.0)
- moved R54 3.52 mm to (187.9, 116.0)
- moved R57 2.61 mm to (186.9, 103.0)
- moved R55 2.08 mm to (187.9, 112.5)
Routing:
- net Net-(C33-Pad2): track 11.8 -> 10.5 mm
Changed lines of the file:
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@@
 	(footprint "104031-0811:MOLEX_104031-0811"
 		(layer "B.Cu")
-		(at 199.875 116.02 90)
+		(at 211.05 115.74 90)
 		(property "Reference" "J9"
 			(at -2.545225 7.385735 90)
@@
 	(footprint "Resistor_SMD:R_0402_1005Metric"
 		(layer "B.Cu")
-		(at 187.24 112.5 180)
+		(at 187.95 115.95 180)
 		(descr "Resistor SMD 0402 (1005 Metric), square (rectangular) end terminal, IPC-7351 nominal, (Body size source: IPC-SM-782 page 72, https://www.pcb-3d.com/wordpress/wp-content/uploads/ipc-sm-782a_amendment_1_and_2.pdf)")
 		(tags "resistor")
@@
 	(footprint "Resistor_SMD:R_0402_1005Metric"
 		(layer "B.Cu")
-		(at 187.24 110.5 180)
+		(at 187.95 112.45 180)
 		(descr "Resistor SMD 0402 (1005 Metric), square (rectangular) end terminal, IPC-7351 nominal, (Body size source: IPC-SM-782 page 72, https://www.pcb-3d.com/wordpress/wp-content/uploads/ipc-sm-782a_amendment_1_and_2.pdf)")
 		(tags "resistor")
@@
 	(footprint "Resistor_SMD:R_0402_1005Metric"
 		(layer "B.Cu")
-		(at 187.49 105.5 180)
+		(at 186.95 102.95 180)
 		(descr "Resistor SMD 0402 (1005 Metric), square (rectangular) end terminal, IPC-7351 nominal, (Body size source: IPC-SM-782 page 72, https://www.pcb-3d.com/wordpress/wp-content/uploads/ipc-sm-782a_amendment_1_and_2.pdf)")
 		(tags "resistor")
@@
 	(footprint "Resistor_SMD:R_0402_1005Metric"
 		(layer "B.Cu")
-		(at 187.24 116 180)
+		(at 188.95 122.95 180)
 		(descr "Resistor SMD 0402 (1005 Metric), square (rectangular) end terminal, IPC-7351 nominal, (Body size source: IPC-SM-782 page 72, https://www.pcb-3d.com/wordpress/wp-content/uploads/ipc-sm-782a_amendment_1_and_2.pdf)")
 		(tags "resistor")
@@
 	(footprint "RFM95W-915S2:XCVR_RFM95W-915S2"
 		(layer "B.Cu")
-		(at 201.55 97.25 180)
+		(at 215.95 90.75 180)
 		(property "Reference" "U6"
 			(at -6.63079 9.54026 0)
@@
 	)
 	(segment
-		(start 125.8875 71.5)
-		(end 127.25 71.5)
-		(width 0.2)
-		(layer "F.Cu")
-		(net "Net-(C33-Pad2)")
-	)
-	(segment
-		(start 128 71.75)
-		(end 128.25 71.5)
-		(width 0.2)
-		(layer "F.Cu")
-		(net "Net-(C33-Pad2)")
-	)
-	(segment
-		(start 128 71.75)
+		(start 128 72.25)
 		(end 128 73.5)
 		(width 0.2)
@@
 	)
 	(segment
-		(start 128.25 71.5)
-		(end 128 71.5)
-		(width 0.2)
-		(layer "F.Cu")
-		(net "Net-(C33-Pad2)")
-	)
-	(segment
-		(start 128 71.5)
-		(end 128 71.75)
+		(start 125.8875 71.5)
+		(end 127.25 71.5)
 		(width 0.2)
 		(layer "F.Cu")
@@
 	(segment
 		(start 134.48 71.5)
-		(end 128.25 71.5)
+		(end 128.75 71.5)
 		(width 0.2)
 		(layer "F.Cu")
@@
 	(segment
 		(start 127.25 71.5)
-		(end 127.75 71.5)
+		(end 128 72.25)
 		(width 0.2)
 		(layer "F.Cu")
@@
 	)
 	(segment
-		(start 127.75 71.5)
-		(end 128 71.75)
-		(width 0.2)
-		(layer "F.Cu")
-		(net "Net-(C33-Pad2)")
-	)
-	(segment
-		(start 128 71.5)
-		(end 127.25 71.5)
+		(start 128.75 71.5)
+		(end 128 72.25)
 		(width 0.2)
 		(layer "F.Cu")
