File: PCE-RCE Carrier/PCE-RCE Carrier.kicad_sch (KiCad schematic)
At the start: 2 parts, among them J5 DF40C-34DP-0.4V_58_, J7 DF40C-34DP-0.4V_58_

Commit message: added payload solenoid gpio, 3v3 rail from power mux to carriers, finished wiring
Connections:
- net +3V3_REG: no longer J5.7
- net +3V3: now reaches J5.3
- net +3V3: now also J5.7
- net PAYLOAD_S: now reaches J5.4
- no-connect marks 27 -> 26
Other:
- sheet Power Distribution and Motor Control ports: added PAYLOAD_SOLENOID; removed none
