File: PCE-RCE Carrier/power_distribution.kicad_sch (KiCad schematic)
At the start: 25 parts, among them J2 XT60PW-F, J3 XT30UPB-M, J4 XT60PW-F, J9 XT30UPB-M, U2 TPS54302DDCR, U3 BD6222HFP-TR, U4 LMR51430, U5 BD6222HFP-TR

Commit message: added payload solenoid gpio, 3v3 rail from power mux to carriers, finished wiring
Parts:
- added J1: Conn_01x02, Connector_PinHeader_2.54mm:PinHeader_1x02_P2.54mm_Vertical, symbol Connector_Generic:Conn_01x02
- added Q1: SP2002KNC, Package_DFN_QFN:Diodes_DFN1006-3, symbol Transistor_FET:SP2002KNC
- added R1: 10k, Resistor_SMD:R_0402_1005Metric, symbol Device:R
Connections:
- net +12V: now also J1.1 (Pin_1)
- net GND: now also Q1.2 (S), R1.2
- new net: J1.2 (Pin_2), Q1.3 (D)
- new net PAYLOAD_SOLENOID: Q1.1 (G), R1.1
Other:
- note added: "Motor Controls"
- note added: "NMOS rated for 20VDS, 0.75A ID"
- note added: "Solenoid Controls"
- note removed: "Motor/Solenoid Controls"

Commit message: DRC changes and updated fab files
Parts:
- added C8: 22u, Capacitor_SMD:C_0805_2012Metric, symbol Device:C
- added C9: 22u 25V, Capacitor_SMD:C_0805_2012Metric, symbol Device:C
- C4: value 44u -> 22u
- C5: value 44u 25V -> 22u 25V
Connections:
- net +12V: now also C9.1
- net +3V3_REG: now also C8.1
- net GND: now also C8.2, C9.2
Other:
- moved on the sheet: C12, C17, C3, C5, L3, R15, R16, R17, R2, R23, U4
