File: RCE Carrier/breakout.kicad_sch (KiCad schematic)
At the start: 3 parts, among them J10 Conn_01x06_Pin, J6 PRT-16766

Commit message: added payload solenoid gpio, 3v3 rail from power mux to carriers, finished wiring
Connections:
- net MOSI: now also J10.5 (Pin_5); no longer J10.3 (Pin_3)
- net SCLK: now also J10.3 (Pin_3); no longer J10.5 (Pin_5)
- net SPI_CS: now also J10.2 (Pin_2); no longer J10.4 (Pin_4)
- net at R42.2: now also J10.4 (Pin_4); no longer J10.2 (Pin_2)
Changed lines of the file:
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@@
+	(wire
+		(pts
+			(xy 132.08 104.14) (xy 123.19 104.14)
+		)
+		(stroke
+			(width 0)
+			(type default)
+		)
+	)
 	(wire
 		(pts
@@
 	(wire
 		(pts
+			(xy 128.27 109.22) (xy 132.08 109.22)
+		)
+		(stroke
+			(width 0)
+			(type default)
+		)
+	)
+	(wire
+		(pts
+			(xy 132.08 111.76) (xy 123.19 111.76)
+		)
+		(stroke
+			(width 0)
+			(type default)
+		)
+	)
+	(wire
+		(pts
+			(xy 132.08 106.68) (xy 123.19 106.68)
+		)
+		(stroke
+			(width 0)
+			(type default)
+		)
+	)
+	(wire
+		(pts
 			(xy 130.81 66.04) (xy 146.05 66.04)
 		)
@@
 	(wire
 		(pts
-			(xy 132.08 111.76) (xy 123.19 111.76)
-		)
-		(stroke
-			(width 0)
-			(type default)
-		)
-	)
-	(wire
-		(pts
-			(xy 132.08 109.22) (xy 123.19 109.22)
-		)
-		(stroke
-			(width 0)
-			(type default)
-		)
-	)
-	(wire
-		(pts
 			(xy 137.16 114.3) (xy 123.19 114.3)
 		)
@@
 	(wire
 		(pts
-			(xy 128.27 104.14) (xy 132.08 104.14)
-		)
-		(stroke
-			(width 0)
-			(type default)
-		)
-	)
-	(wire
-		(pts
 			(xy 123.19 101.6) (xy 144.78 101.6)
 		)
@@
 	(wire
 		(pts
-			(xy 132.08 106.68) (xy 123.19 106.68)
-		)
-		(stroke
-			(width 0)
-			(type default)
-		)
-	)
-	(wire
-		(pts
 			(xy 146.05 66.04) (xy 146.05 67.31)
 		)
@@
 			(width 0)
 			(type default)
-		)
-	)
-	(hierarchical_label "MOSI"
-		(shape input)
-		(at 132.08 106.68 0)
-		(effects
-			(font
-				(size 1.27 1.27)
-			)
-			(justify left)
-		)
-	)
-	(hierarchical_label "MISO"
-		(shape output)
-		(at 132.08 104.14 0)
-		(effects
-			(font
-				(size 1.27 1.27)
-			)
-			(justify left)
 		)
 	)
@@
 		)
 	)
+	(hierarchical_label "MISO"
+		(shape output)
+		(at 132.08 109.22 0)
+		(effects
+			(font
+				(size 1.27 1.27)
+			)
+			(justify left)
+		)
+	)
 	(hierarchical_label "SCLK"
+		(shape input)
+		(at 132.08 106.68 0)
+		(effects
+			(font
+				(size 1.27 1.27)
+			)
+			(justify left)
+		)
+	)
+	(hierarchical_label "SCL"
+		(shape input)
+		(at 134.62 58.42 0)
+		(effects
+			(font
+				(size 1.27 1.27)
+			)
+			(justify left)
+		)
+	)
+	(hierarchical_label "MOSI"
 		(shape input)
 		(at 132.08 111.76 0)
@@
 	(hierarchical_label "SPI_CS"
 		(shape input)
-		(at 132.08 109.22 0)
-		(effects
-			(font
-				(size 1.27 1.27)
-			)
-			(justify left)
-		)
-	)
-	(hierarchical_label "SCL"
-		(shape input)
-		(at 134.62 58.42 0)
+		(at 132.08 104.14 0)
 		(effects
 			(font
@@
 	(symbol
 		(lib_id "Device:R_Small")
-		(at 125.73 104.14 270)
+		(at 125.73 109.22 270)
 		(mirror x)
 		(unit 1)
@@
 		(dnp no)
 		(property "Reference" "R42"
-			(at 130.048 104.14 90)
+			(at 130.048 109.22 90)
 			(show_name no)
 			(do_not_autoplace no)
@@
 		)
 		(property "Value" "22"
-			(at 125.73 104.14 90)
+			(at 125.73 109.22 90)
 			(show_name no)
 			(do_not_autoplace no)
@@
 		)
 		(property "Footprint" "Resistor_SMD:R_0402_1005Metric"
-			(at 125.73 104.14 0)
+			(at 125.73 109.22 0)
 			(hide yes)
 			(show_name no)
@@
 		)
 		(property "Datasheet" ""
-			(at 125.73 104.14 0)
+			(at 125.73 109.22 0)
 			(hide yes)
 			(show_name no)
@@
 		)
 		(property "Description" "Resistor, small symbol"
-			(at 125.73 104.14 0)
-			(hide yes)
-			(show_name no)
+			(at 125.73 109.22 0)
+			(hide yes)
+			(show_name no)

Commit message: DRC changes and updated fab files
Parts:
- J10: footprint Connector_PinSocket_2.54mm:PinSocket_1x06_P2.54mm_Vertical -> Connector_PinHeader_2.54mm:PinHeader_1x06_P2.54mm_Vertical
Changed lines of the file:
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@@
 			)
 		)
-		(property "Footprint" "Connector_PinSocket_2.54mm:PinSocket_1x06_P2.54mm_Vertical"
+		(property "Footprint" "Connector_PinHeader_2.54mm:PinHeader_1x06_P2.54mm_Vertical"
 			(at 118.11 106.68 0)
 			(hide yes)
