File: ACE Carrier/ACE Carrier.kicad_pcb (KiCad board)
At the start: 2 copper layers, 39 parts, among them J1 Conn_01x04, J10 Conn_01x06_Pin, J2 XT60PW-F, J3 XT60PW-F, J4 XT60PW-F, J5 DF40C-34DP-0.4V_58_, J6 PRT-16766, J7 DF40C-34DP-0.4V_58_, J8 Conn_01x03, U1 NCP1117-5.0_SOT223, U2 TPS54302DDCR, U3 ADXL345, U4 TPS62130

Commit message: update ace carrier interface pinout + initial layout
Parts:
- removed D1, D2: RB496EATR, RB496EATR:DIO_FTZ_ROM
- removed J4: XT60PW-F, XT60PW-F:AMASS_XT60PW-F
- added C14: 22u, Capacitor_SMD:C_0805_2012Metric, F.Cu at (164.0, 72.2)
- added R7: 10k, Resistor_SMD:R_0402_1005Metric, F.Cu at (124.5, 80.5)
- added R8: 10k, Resistor_SMD:R_0402_1005Metric, F.Cu at (124.5, 82.5)
- C4: value 44u -> 22u
- J1: footprint Connector_JST:JST_PH_S4B-PH-K_1x04_P2.00mm_Horizontal -> Connector_JST:JST_PH_B4B-PH-K_1x04_P2.00mm_Vertical
- J2, J3: value XT60PW-F -> XT30UPB-M; footprint XT60PW-F:AMASS_XT60PW-F -> XT30UPB-M:AMASS_XT30UPB-M
- J5, J7: moved to B.Cu
- R16: value 22.1k -> 22.1k 1%
- R2: value 100k -> 100k 1%
- R23: value 49.9k -> 49.9 1%
- moved C12 110.4 mm to (238.7, 81.2)
- moved R4 105.4 mm to (235.7, 93.7)
- moved R5 105.4 mm to (235.7, 96.2)
- moved R6 105.4 mm to (235.7, 98.8)
- moved L1 101.5 mm to (224.5, 100.5)
- moved C10 93.5 mm to (219.5, 97.5)
- moved C13 93.5 mm to (219.5, 103.5)
- moved C7 93.5 mm to (219.5, 94.5)
- moved U4 88.7 mm to (206.8, 116.0)
- moved U1 84.3 mm to (197.1, 70.0)
- moved J1 58.1 mm to (182.2, 61.5), turned to 90 degrees
- moved J2 55.5 mm to (152.0, 84.8), turned to -90 degrees
- moved J5 55.3 mm to (169.5, 57.2), turned to 0 degrees
- moved C4 52.8 mm to (166.2, 72.2), turned to -90 degrees
- moved J3 51.8 mm to (152.0, 70.8), turned to 90 degrees
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Connections:
- net /Airbrakes Sensors/PITOT_SIGNAL_5V renamed /Airbrakes Sensors/PITOT_SGL_5V
- net /PITOT_SIGNAL renamed /PITOT_SGL
- C11 pad 2: +3V3_REG -> Net-(U2-SW)
- C6 pad 1: +5V_REG -> +5V
- J10 pad 2: /MOSI -> Net-(J10-Pin_2)
- J10 pad 3: Net-(J10-Pin_3) -> /MOSI
- J5 pad 1: unconnected-(J5-Pad1) -> GND
- J5 pad 10: unconnected-(J5-Pad10) -> /SCL
- J5 pad 11: unconnected-(J5-Pad11) -> GND
- J5 pad 25: unconnected-(J5-Pad25) -> GND
- J5 pad 3: unconnected-(J5-Pad3) -> +3V3
- J5 pad 7: +3V3_REG -> +3V3
- J5 pad 8: unconnected-(J5-Pad8) -> /SDA
- J5 pad 9: unconnected-(J5-Pad9) -> GND
- J7 pad 1: unconnected-(J7-Pad1) -> GND
- J7 pad 12: unconnected-(J7-Pad12) -> +3V3_REG
- J7 pad 16: unconnected-(J7-Pad16) -> +3V3_REG
- J7 pad 2: unconnected-(J7-Pad2) -> GND
- J7 pad 20: unconnected-(J7-Pad20) -> +3V3_REG
- J7 pad 24: unconnected-(J7-Pad24) -> +3V3_REG
- J7 pad 27: /SDA -> unconnected-(J7-Pad27)
- J7 pad 28: unconnected-(J7-Pad28) -> +3V3_REG
- J7 pad 29: /SCL -> unconnected-(J7-Pad29)
- J7 pad 32: unconnected-(J7-Pad32) -> GND
- J7 pad 34: unconnected-(J7-Pad34) -> GND
- J7 pad 7: unconnected-(J7-Pad7) -> GND
- J7 pad 8: +3V3_REG -> unconnected-(J7-Pad8)
- R47 pad 2: Net-(J10-Pin_3) -> Net-(J10-Pin_2)
- U1 pad 2: +5V_REG -> +5V
Other:
- board outline added: 38 x 39.5 mm

Commit message: initial ace routing
Parts:
- C12: footprint Capacitor_SMD:C_0402_1005Metric -> Capacitor_SMD:C_0805_2012Metric
- moved C5 93.4 mm to (174.8, 73.6), turned to 180 degrees
- moved R6 88.8 mm to (158.0, 55.6), turned to -90 degrees
- moved C6 88.4 mm to (174.8, 71.0), turned to 180 degrees
- moved C12 87.4 mm to (155.1, 55.6)
- moved R5 86.2 mm to (159.6, 55.6), turned to 90 degrees
- moved R4 83.7 mm to (161.2, 55.6), turned to 90 degrees
- moved C10 78.9 mm to (151.6, 57.2), turned to 90 degrees
- moved J10 77.4 mm to (184.2, 89.8), turned to 180 degrees
- moved U4 76.3 mm to (155.8, 59.3), turned to 180 degrees
- moved L1 75.8 mm to (160.6, 59.8), turned to -90 degrees
- moved C7 75.6 mm to (151.6, 61.2), turned to -90 degrees
- moved C13 74.1 mm to (157.0, 63.6), turned to 180 degrees
- moved J8 69.4 mm to (165.2, 65.4)
- moved R47 67.8 mm to (181.1, 87.2)
- moved U3 57.2 mm to (170.8, 81.4), turned to -90 degrees
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Connections:
- J10 pad 4: /SPI_CS -> /SCLK
- J10 pad 5: /SCLK -> /SPI_CS
- J6 pad 5: (no net) -> GND
- J6 pad 6: (no net) -> GND
Routing:
- net GND: track 0.00 -> 62.6 mm, vias 0 -> 18
- net /SDA: track 0.00 -> 39.4 mm, vias 0 -> 1
- net /ADXL_INT2: track 0.00 -> 31.1 mm, vias 0 -> 1
- net /SCL: track 0.00 -> 29.7 mm, vias 0 -> 1
- net VIN: track 0.00 -> 27.6 mm, vias 0 -> 2
- net /ADXL_INT1: track 0.00 -> 27.1 mm, vias 0 -> 1
- net /SPI_CS: track 0.00 -> 19.1 mm
- net /SCLK: track 0.00 -> 17.5 mm
- net /MOSI: track 0.00 -> 15.7 mm
- net /PITOT_SGL: track 0.00 -> 14.6 mm, vias 0 -> 1
- net Net-(U2-SW): track 0.00 -> 13.6 mm, vias 0 -> 3
- net +6V: track 0.00 -> 12.8 mm, vias 0 -> 2
- net /MISO: track 0.00 -> 12.0 mm, vias 0 -> 1
- net Net-(J2-PadP): track 0.00 -> 9.00 mm
- net +3V3: track 0.00 -> 8.50 mm, vias 0 -> 4
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- added copper zone on F.Cu, net +3V3
- added copper zone on F.Cu, net +3V3_REG
- added copper zone on F.Cu, net +5V
- added copper zone on F.Cu, net +6V
- added copper zone on B.Cu, net GND
- added copper zone on F.Cu, net Net-(L1-Pad1)
- added copper zone on F.Cu, net VIN

Commit message: silkscreen shenanigans
Parts:
- added G***: LOGO, WURocketry_logo:WURocketry_logo, B.Cu at (177.6, 64.0)
- J10: footprint Connector_PinSocket_2.54mm:PinSocket_1x06_P2.54mm_Vertical -> Connector_PinHeader_2.54mm:PinHeader_1x06_P2.54mm_Vertical
Connections:
- J6 pad 5: GND -> (no net)
- J6 pad 6: GND -> (no net)
Other:
- board text added: "+6V"
- board text added: "3V3"
- board text added: "3V3 BUCK"
- board text added: "5V"
- board text added: "6V BUCK"
- board text added: "ACE"
- board text added: "ADXL"
- board text added: "BAT"
- board text added: "CS"
- board text added: "Carrier"
- board text added: "Department of Electrical and Systems Engineering Washington University in St. Louis"
- board text added: "GND"
- board text added: "LDO"
- board text added: "MISO"
- board text added: "MOSI"
- board text added: "PITOT TUBE"
- board text added: "PWM"
- board text added: "QWIIC I2C"
- board text added: "SCK"
- board text added: "SERVO"
- board text added: "SIGNAL"
- board text added: "SWITCH"
- board text added: "WURocketry 2026-2027"
- board text added: "for Airdahl Flight Computer"
- board text added: "spring break - airbrake - ?"
- board text added: "this is a haiku we should cut the payload team live laugh love rocket"
- board text added: "{dblquote}a lot of things were said, and i don't remember most of them{dblquote}"
- board text added: "{dblquote}i find going in easier{dblquote}"
- board text added: "{dblquote}i'm calling this the baby test because you shake it{dblquote}"
- board text added: "{dblquote}set analog pin to high{dblquote}"
- board text added: "{dblquote}we can always code in the car{dblquote}"
- board text added: "{dblquote}we can epoxy it in{dblquote}"
- board text added: "{dblquote}what a dumb question 'did it work?'{dblquote}"
